File: hardware/picostepseq_mk2_16.brd (EAGLE design)
At the start: 152.4 x 82.5 mm, 55 parts, among them J1 SJ-3523-SMT, J2 SJ-3523-SMT, SW1 LED_SWITCHSTEP, SW10 LED_SWITCHSTEP, SW11 LED_SWITCHSTEP, SW12 LED_SWITCHSTEP, SW13 LED_SWITCHSTEP, SW14 LED_SWITCHSTEP, SW15 LED_SWITCHSTEP, SW16 LED_SWITCHSTEP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

Commit message: "finish" picostepseq_mk2_16
Parts:
- moved R4 29.5 mm to (120.7, 67.3), turned to 180 degrees
- moved U2 19.7 mm to (120.7, 59.7), turned to 90 degrees
- moved S1 13.3 mm to (102.9, 54.6), turned to 180 degrees
- moved C1 11.7 mm to (120.7, 52.1), turned to 180 degrees
- moved ENC1 10.5 mm to (103.4, 69.6)
- moved R1 3.81 mm to (131.4, 71.6)
- moved R2 3.81 mm to (131.4, 69.1)
- moved J1 3.81 mm to (152.9, 71.0)
- moved J2 3.81 mm to (152.9, 54.9)
- moved R3 1.27 mm to (132.1, 53.3)
- renumbered D20 to D19
Connections:
- net ROTSW: now also U1.29, U1.P$29; no longer U1.34, U1.P$34
- net SW0: now also U1.34, U1.P$34; no longer U1.29, U1.P$29
Routing:
- net ROTSW: track 106.9 -> 84.1 mm
- net N$2: track 31.1 -> 8.44 mm
- net N$4: track 42.6 -> 23.4 mm
- net SW0: track 72.7 -> 91.6 mm
- net MIDI_IN: track 71.0 -> 86.9 mm
- net ROTA: track 101.7 -> 88.9 mm
- net ROTB: track 90.9 -> 78.9 mm
- net COL5: track 163.8 -> 169.2 mm
- net N$1: track 5.85 -> 10.6 mm
- net N$14: track 12.7 -> 17.0 mm
- net N$13: track 15.9 -> 18.2 mm
- net LED9: track 116.9 -> 118.4 mm
- net ROW4: track 187.6 -> 188.9 mm
- net COL1: track 140.4 -> 139.2 mm
- net COL2: track 153.4 -> 152.2 mm
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Other:
- board size 152.4 x 82.5 mm -> 156.2 x 82.5 mm
- board text added: "D1-D19: 1N4148"
- board text removed: "D1-D18: 1N4148"
