File: hardware/picostepseq_mk2_16.sch (EAGLE design)
At the start: 55 parts, among them J1 SJ-3523-SMT, J2 SJ-3523-SMT, SW1 LED_SWITCHSTEP, SW10 LED_SWITCHSTEP, SW11 LED_SWITCHSTEP, SW12 LED_SWITCHSTEP, SW13 LED_SWITCHSTEP, SW14 LED_SWITCHSTEP, SW15 LED_SWITCHSTEP, SW16 LED_SWITCHSTEP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

Commit message: "finish" picostepseq_mk2_16
Parts:
- renumbered D20 to D19
Connections:
- net ROTSW: now also U1.GP22; no longer U1.GP28
- net SW0: now also U1.GP28; no longer U1.GP22
